File: PCB/board/plat_board/plat_board.kicad_pcb (KiCad board)
At the start: 2 copper layers, 95 x 94.9 mm, 37 parts, among them J1 Step_Select1, J10 VIN, J11 STM32F4, J12 STM32F4, J13 Btn_OnOff, J14 Conn_Ext2, J15 FSR, J16 VS3, J17 MPU, J18 VS1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

Commit message: Adding image
Routing:
- net GND: track 4.47 -> 0.08 mm, vias 1 -> 37
- net /M2_DIR: track 61.6 -> 62.9 mm
Other:
- board text added: "STM32F401"
- board text added: "Vin"
- board text removed: "Vin - J4"
